File: Nexus 01 schematic.kicad_pcb (KiCad board)
At the start: 4 copper layers, 48 parts, among them J1 Conn_01x02_Male, J2 Conn_01x02_Male, J3 Conn_01x02_Male, J4 Conn_01x02_Male, J5 USB_C_Receptacle_USB2.0, J6 Conn_01x02_Male, Q1 SI2302, Q2 SI2302, Q3 SI2302, Q4 SI2302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

Commit message: Add files via upload
Parts:
- moved C8 119.0 mm to (91.6, 49.8), turned to -90 degrees
- moved U2 116.2 mm to (95.0, 67.6)
- moved C3 115.4 mm to (93.6, 49.7), turned to -90 degrees
- moved D6 101.9 mm to (114.6, 68.8)
- moved D8 95.3 mm to (121.4, 74.0)
- moved SW2 92.3 mm to (94.2, 78.6)
- moved J6 90.9 mm to (126.8, 73.0), turned to 90 degrees
- moved U6 90.7 mm to (126.3, 70.0)
- moved Q1 89.8 mm to (128.3, 49.2)
- moved Q2 89.5 mm to (128.4, 52.5)
- moved Q3 89.2 mm to (128.6, 56.0)
- moved Q4 89.0 mm to (128.7, 59.4)
- moved D7 88.8 mm to (127.0, 78.2)
- moved J4 85.0 mm to (130.4, 62.6), turned to -90 degrees
- moved D4 85.0 mm to (133.0, 51.6)
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Routing:
- net GND: track 0.00 -> 276.0 mm, vias 0 -> 19
- net +3V3: track 0.00 -> 112.2 mm, vias 0 -> 6
- net /VBAT: track 0.00 -> 93.3 mm, vias 0 -> 8
- net GPIO1: track 0.00 -> 83.2 mm, vias 0 -> 4
- net GPIO2: track 0.00 -> 81.0 mm, vias 0 -> 2
- net EN: track 0.00 -> 75.3 mm, vias 0 -> 4
- net GPIO0: track 0.00 -> 51.4 mm, vias 0 -> 3
- net MOTOR4: track 0.00 -> 43.4 mm, vias 0 -> 2
- net MOTOR3: track 0.00 -> 40.3 mm, vias 0 -> 1
- net GPIO19: track 0.00 -> 34.3 mm, vias 0 -> 2
- net MOTOR1: track 0.00 -> 30.6 mm
- net MOTOR2: track 0.00 -> 30.5 mm, vias 0 -> 2
- net +5V: track 0.00 -> 29.9 mm
- net Net-(D4-A): track 0.00 -> 26.5 mm, vias 0 -> 1
- net GPIO12: track 0.00 -> 21.3 mm, vias 0 -> 2
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Other:
- board outline added: 48.1 x 35 mm
- board text added: "C2"
- board text added: "Routed by: Traffic Person Made by: Rohan"
